File: Breadboard Power Supply.kicad_pcb (KiCad board)
At the start: 2 copper layers, 0 parts

Commit message: Update PCB Design
Parts:
- added C1: 10u, Capacitor_THT:C_Disc_D3.0mm_W1.6mm_P2.50mm, F.Cu at (139.3, 79.2)
- added C2: 0u1, Capacitor_THT:C_Disc_D3.0mm_W1.6mm_P2.50mm, F.Cu at (131.9, 79.2)
- added C3: 1u, Capacitor_THT:C_Disc_D3.0mm_W1.6mm_P2.50mm, F.Cu at (132.9, 109.5)
- added D1: LED, LED_THT:LED_D5.0mm, F.Cu at (152.0, 94.7)
- added J1: Conn_01x02_Pin, Connector_PinHeader_2.54mm:PinHeader_1x02_P2.54mm_Vertical, F.Cu at (161.1, 70.4)
- added J2: Conn_01x02_Pin, Connector_PinHeader_2.54mm:PinHeader_1x02_P2.54mm_Vertical, F.Cu at (161.1, 116.1)
- added J5: Screw_Terminal_01x02, TerminalBlock:TerminalBlock_bornier-2_P5.08mm, F.Cu at (148.2, 72.6)
- added J6: Screw_Terminal_01x02, TerminalBlock:TerminalBlock_bornier-2_P5.08mm, F.Cu at (148.2, 116.8)
- added J7: Barrel_Jack_Switch, Connector_BarrelJack:BarrelJack_Horizontal, F.Cu at (143.5, 93.5)
- added R1: 330, Resistor_THT:R_Axial_DIN0204_L3.6mm_D1.6mm_P7.62mm_Horizontal, F.Cu at (147.2, 87.1)
- added R2: 330, Resistor_THT:R_Axial_DIN0204_L3.6mm_D1.6mm_P7.62mm_Horizontal, F.Cu at (154.8, 103.4)
- added R3: 560, Resistor_THT:R_Axial_DIN0204_L3.6mm_D1.6mm_P7.62mm_Horizontal, F.Cu at (147.1, 106.7)
- added REF**: KiCad-Logo2_5mm_SilkScreen, Symbol:KiCad-Logo2_5mm_SilkScreen, B.Cu at (150.9, 104.7)
- added S1: EG1218, EG1218 SPDT Switch:SW_EG1218, F.Cu at (136.2, 71.1)
- added S2: EG1218, EG1218 SPDT Switch:SW_EG1218, F.Cu at (136.2, 118.4)
- added SW1: SW_Wuerth_450301014042, Button_Switch_THT:SW_Slide-03_Wuerth-WS-SLTV_10x2.5x6.4_P2.54mm, F.Cu at (151.0, 81.5)
- added U1: LM7805_TO220, Package_TO_SOT_THT:TO-220-3_Vertical, F.Cu at (137.0, 83.4)
- added U2: LM317_TO-220, Package_TO_SOT_THT:TO-220-3_Vertical, F.Cu at (131.9, 104.9)
Routing:
- net /PWR_output: track 0.00 -> 104.7 mm
- net /3.3V: track 0.00 -> 66.9 mm, vias 0 -> 1
- net /5V: track 0.00 -> 56.5 mm
- net /12V: track 0.00 -> 52.3 mm
- net Net-(U2-ADJ): track 0.00 -> 29.9 mm
- net /PWR_input: track 0.00 -> 16.9 mm
- net Net-(D1-A): track 0.00 -> 7.68 mm
- added copper zone on B.Cu, net GND
Other:
- board outline added: 35.3 x 53.3 mm
- board text added: "+"
- board text added: "-"
- board text added: "3.3V"
- board text added: "5V"
- board text added: "Breadboard Power Supply"
- board text added: "GND"
- board text added: "Henry Munachimso"
- board text added: "OFF"
- board text added: "ON"
- board text added: "v1.0"
