File: Breadboard Power Supply.kicad_pcb (KiCad board)
At the start: 2 copper layers, 35.3 x 53.3 mm, 18 parts, among them J1 Conn_01x02_Pin, J2 Conn_01x02_Pin, J5 Screw_Terminal_01x02, J6 Screw_Terminal_01x02, J7 Barrel_Jack_Switch, SW1 SW_Wuerth_450301014042, U1 LM7805_TO220, U2 LM317_TO-220

Commit message: Fix bug in schematic
Connections:
- J1 pad 2: /PWR_output -> /PWR_OUT_TOP
- J2 pad 2: /PWR_output -> /PWR_OUT_DOWN
- J5 pad 2: /PWR_output -> /PWR_OUT_TOP
- J6 pad 2: /PWR_output -> /PWR_OUT_DOWN
- S1 pad 2: /PWR_output -> /PWR_OUT_TOP
- S2 pad 2: /PWR_output -> /PWR_OUT_DOWN
Routing:
- net /PWR_output: track 104.7 -> 0.00 mm
- net (no net): track 0.00 -> 48.4 mm
- net /PWR_OUT_DOWN: track 0.00 -> 28.3 mm
- net /PWR_OUT_TOP: track 0.00 -> 26.0 mm
Changed lines of the file:
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@@
 		(title "Breadboard Power Supply")
 		(date "2025-09-23")
-		(rev "v1.0")
+		(rev "v2.0")
 	)
 	(layers
@@
 	(net 4 "/3.3V")
 	(net 5 "Net-(D1-A)")
-	(net 6 "/PWR_output")
+	(net 6 "/PWR_OUT_TOP")
 	(net 7 "/PWR_input")
 	(net 8 "Net-(U2-ADJ)")
 	(net 9 "unconnected-(SW1-C-Pad2)")
+	(net 10 "/PWR_OUT_DOWN")
 	(footprint "Capacitor_THT:C_Disc_D3.0mm_W1.6mm_P2.50mm"
 		(locked yes)
@@
 			(layers "*.Cu" "*.Mask")
 			(remove_unused_layers no)
-			(net 6 "/PWR_output")
+			(net 6 "/PWR_OUT_TOP")
 			(pinfunction "Pin_2")
 			(pintype "passive")
@@
 			(layers "*.Cu" "*.Mask")
 			(remove_unused_layers no)
-			(net 6 "/PWR_output")
+			(net 6 "/PWR_OUT_TOP")
 			(pinfunction "Pin_2")
 			(pintype "passive")
@@
 			(layers "*.Cu" "*.Mask")
 			(remove_unused_layers no)
-			(net 6 "/PWR_output")
+			(net 10 "/PWR_OUT_DOWN")
 			(pinfunction "Pin_2")
 			(pintype "passive")
@@
 			(layers "*.Cu" "*.Mask")
 			(remove_unused_layers no)
-			(net 6 "/PWR_output")
+			(net 10 "/PWR_OUT_DOWN")
 			(pinfunction "Pin_2")
 			(pintype "passive")
@@
 			(layers "*.Cu" "*.Mask")
 			(remove_unused_layers no)
-			(net 6 "/PWR_output")
+			(net 10 "/PWR_OUT_DOWN")
 			(pintype "passive")
 			(solder_mask_margin 0.102)
@@
 			(layers "*.Cu" "*.Mask")
 			(remove_unused_layers no)
-			(net 6 "/PWR_output")
+			(net 6 "/PWR_OUT_TOP")
 			(pintype "passive")
 			(solder_mask_margin 0.102)
@@
 	)
 	(segment
+		(start 152.2476 116.84)
+		(end 153.2636 116.84)
+		(width 0.35)
+		(locked yes)
+		(layer "F.Cu")
+		(net 0)
+	)
+	(segment
+		(start 157.0736 109.22)
+		(end 153.2636 113.03)
+		(width 0.35)
+		(locked yes)
+		(layer "F.Cu")
+		(net 0)
+	)
+	(segment
+		(start 153.2636 72.644)
+		(end 153.2636 74.676)
+		(width 0.35)
+		(locked yes)
+		(layer "F.Cu")
+		(net 0)
+	)
+	(segment
+		(start 153.2636 113.03)
+		(end 153.2636 116.84)
+		(width 0.35)
+		(locked yes)
+		(layer "F.Cu")
+		(net 0)
+	)
+	(segment
+		(start 157.0736 78.486)
+		(end 157.0736 109.22)
+		(width 0.35)
+		(locked yes)
+		(layer "F.Cu")
+		(net 0)
+	)
+	(segment
+		(start 153.2636 74.676)
+		(end 157.0736 78.486)
+		(width 0.35)
+		(locked yes)
+		(layer "F.Cu")
+		(net 0)
+	)
+	(segment
 		(start 154.7876 86.106)
 		(end 154.7876 87.122)
@@
 	)
 	(segment
-		(start 136.2056 71.12)
-		(end 137.7296 69.596)
+		(start 137.8204 69.5052)
+		(end 137.8204 69.3928)
 		(width 0.35)
-		(locked yes)
 		(layer "F.Cu")
 		(net 6)
 	)
 	(segment
-		(start 150.2156 120.142)
-		(end 150.2156 118.872)
-		(width 0.35)
-		(locked yes)
-		(layer "F.Cu")
-		(net 6)
-	)
-	(segment
-		(start 153.2636 72.644)
-		(end 158.8516 72.644)
-		(width 0.35)
-		(locked yes)
-		(layer "F.Cu")
-		(net 6)
-	)
-	(segment
-		(start 150.2156 118.872)
-		(end 152.2476 116.84)
-		(width 0.35)
-		(locked yes)
-		(layer "F.Cu")
-		(net 6)
-	)
-	(segment
-		(start 136.2056 118.364)
-		(end 136.2056 119.594)
-		(width 0.35)
-		(locked yes)
-		(layer "F.Cu")
-		(net 6)
-	)
-	(segment
-		(start 152.2476 116.84)
-		(end 153.2636 116.84)
-		(width 0.35)
-		(locked yes)
-		(layer "F.Cu")
-		(net 6)
-	)
-	(segment
-		(start 137.7296 69.596)
-		(end 152.2476 69.596)
-		(width 0.35)
-		(locked yes)
-		(layer "F.Cu")
-		(net 6)
-	)
-	(segment
-		(start 153.2636 116.84)
-		(end 155.8036 116.84)
-		(width 0.35)
-		(locked yes)
-		(layer "F.Cu")
-		(net 6)
-	)
-	(segment
-		(start 159.1106 72.893)
-		(end 161.1376 72.893)
-		(width 0.35)
-		(locked yes)
-		(layer "F.Cu")
-		(net 6)
-	)
-	(segment
-		(start 157.0736 109.22)
-		(end 153.2636 113.03)
-		(width 0.35)
-		(locked yes)
-		(layer "F.Cu")
-		(net 6)
-	)
-	(segment
-		(start 157.6324 118.6688)
-		(end 161.1376 118.6688)
-		(width 0.35)
-		(locked yes)
-		(layer "F.Cu")
-		(net 6)
-	)
-	(segment
-		(start 155.8036 116.84)
-		(end 157.6324 118.6688)
-		(width 0.35)
-		(locked yes)
-		(layer "F.Cu")
-		(net 6)
-	)
-	(segment
-		(start 159.1056 72.898)
-		(end 159.1106 72.893)
-		(width 0.35)
-		(locked yes)
-		(layer "F.Cu")
-		(net 6)
-	)
-	(segment
-		(start 153.2636 72.644)
-		(end 153.2636 74.676)
-		(width 0.35)
-		(locked yes)
-		(layer "F.Cu")
-		(net 6)
-	)
-	(segment
-		(start 136.2056 119.594)
-		(end 136.7536 120.142)
-		(width 0.35)
-		(locked yes)
-		(layer "F.Cu")
-		(net 6)
-	)
-	(segment
-		(start 158.8516 72.644)
-		(end 159.1056 72.898)
-		(width 0.35)
-		(locked yes)
-		(layer "F.Cu")
-		(net 6)
-	)
-	(segment
-		(start 153.2636 113.03)
-		(end 153.2636 116.84)
-		(width 0.35)
-		(locked yes)
-		(layer "F.Cu")
-		(net 6)
-	)
-	(segment
-		(start 157.0736 78.486)
-		(end 157.0736 109.22)
+		(start 136.2056 71.12)
+		(end 137.8204 69.5052)
 		(width 0.35)
-		(locked yes)
 		(layer "F.Cu")
 		(net 6)
 	)
 	(segment
-		(start 153.2636 74.676)
-		(end 157.0736 78.486)
+		(start 137.8204 69.3928)
+		(end 150.0124 69.3928)
 		(width 0.35)
-		(locked yes)
 		(layer "F.Cu")
 		(net 6)
 	)
 	(segment
-		(start 153.2636 70.612)
-		(end 153.2636 72.644)
+		(start 154.1136 72.893)
+		(end 153.8646 72.644)
 		(width 0.35)
-		(locked yes)
 		(layer "F.Cu")
 		(net 6)
 	)
 	(segment
-		(start 152.2476 69.596)
-		(end 153.2636 70.612)
+		(start 150.0124 69.3928)
+		(end 152.838629 72.219029)
 		(width 0.35)
-		(locked yes)
 		(layer "F.Cu")
 		(net 6)
 	)
 	(segment
-		(start 136.7536 120.142)
-		(end 150.2156 120.142)
+		(start 161.1376 72.893)
+		(end 154.1136 72.893)
 		(width 0.35)
-		(locked yes)
 		(layer "F.Cu")
 		(net 6)
@@
 		(net 8)
 	)
+	(segment
+		(start 153.2636 117.7544)
+		(end 153.2636 117.441)
+		(width 0.35)
+		(layer "F.Cu")
+		(net 10)
+	)
+	(segment
+		(start 160.3248 119.4816)
+		(end 154.9908 119.4816)
+		(width 0.35)
+		(layer "F.Cu")
+		(net 10)
+	)
+	(segment
+		(start 150.969 119.7356)
+		(end 153.2636 117.441)
+		(width 0.35)
+		(layer "F.Cu")
+		(net 10)
+	)
+	(segment
+		(start 136.2056 119.1368)
+		(end 136.8044 119.7356)
+		(width 0.35)
+		(layer "F.Cu")
+		(net 10)
+	)
+	(segment
+		(start 136.2056 118.364)
+		(end 136.2056 119.1368)
+		(width 0.35)
+		(layer "F.Cu")
+		(net 10)
+	)
+	(segment
+		(start 161.1376 118.6688)
+		(end 160.3248 119.4816)
+		(width 0.35)
+		(layer "F.Cu")
+		(net 10)
+	)
+	(segment
+		(start 136.8044 119.7356)
+		(end 150.969 119.7356)
+		(width 0.35)
+		(layer "F.Cu")
+		(net 10)
+	)
+	(segment
+		(start 154.9908 119.4816)
+		(end 153.2636 117.7544)
+		(width 0.35)
+		(layer "F.Cu")
+		(net 10)
+	)
 	(zone
