File: Breadboard Power Supply.kicad_pcb (KiCad board)
At the start: 2 copper layers, 35.3 x 53.3 mm, 18 parts, among them J1 Conn_01x02_Pin, J2 Conn_01x02_Pin, J5 Screw_Terminal_01x02, J6 Screw_Terminal_01x02, J7 Barrel_Jack_Switch, SW1 SW_Wuerth_450301014042, U1 LM7805_TO220, U2 LM317_TO-220

Commit message: Fix issue with power flag
Routing:
- net (no net): track 48.4 -> 0.00 mm
- net /PWR_OUT_DOWN: track 28.3 -> 29.3 mm
